Commit message: Add quad RL package and trained baselines

File: URDF_description/urdf/URDF_quad.urdf (robot description, URDF)
Before this commit: robot insectoid_mini_quad, 19 links, 18 joints
Links:
- added link BL_FOOT, mass 0.02; collision sphere radius=0.018; visual sphere radius=0.018
- added link BR_FOOT, mass 0.02; collision sphere radius=0.018; visual sphere radius=0.018
- added link ML_FOOT, mass 0.02; collision sphere radius=0.018; visual sphere radius=0.018
- added link MR_FOOT, mass 0.02; collision sphere radius=0.018; visual sphere radius=0.018
Joints:
- added joint BL_foot_fixed_joint: type fixed, parent BL_tibia_1, child BL_FOOT, origin xyz=-0.2 0 0.069 rpy=0 0 0
- added joint BR_foot_fixed_joint: type fixed, parent BR_tibia_1, child BR_FOOT, origin xyz=0.2 0 -0.069 rpy=0 0 0
- added joint ML_foot_fixed_joint: type fixed, parent ML_tibia_1, child ML_FOOT, origin xyz=-0.2 0 0.069 rpy=0 0 0
- added joint MR_foot_fixed_joint: type fixed, parent MR_tibia_1, child MR_FOOT, origin xyz=0.2 0 -0.069 rpy=0 0 0
- joint FL_coxa_joint: origin xyz=-0.08 0.14 -0.002 rpy=3.141592651 2.538366994e-09 0.7853981634 -> xyz=-0.08 0.14 -0.002 rpy=3.141592652 -3.108851958e-09 -1.047197551
- joint FR_coxa_joint: origin xyz=0.08 0.14 -0.002 rpy=0 -0 0.7853981634 -> xyz=0.08 0.14 -0.002 rpy=0 -0 1.047197551
